File: check_in_wizard/check_in_wizard.kicad_sch (KiCad schematic)
At the start: 2 parts, among them U1 STM32F103C8Tx

Commit message: test macos
Parts:
- added U2: IR4301, Package_DFN_QFN:Infineon_PQFN-22-15-4EP_6x5mm_P0.65mm, symbol Amplifier_Audio:IR4301
Connections:
- new net: U2.15 (COM), U2.9 (COM)
Changed lines of the file:
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@@
+    )
+  )
+  (symbol (lib_id "Amplifier_Audio:IR4301") (at 44.45 83.82 0) (unit 1)
+    (in_bom yes) (on_board yes) (dnp no) (fields_autoplaced)
+    (property "Reference" "U2" (at 51.7241 60.96 0)
+      (effects (font (size 1.27 1.27)) (justify left))
+    )
+    (property "Value" "IR4301" (at 51.7241 63.5 0)
+      (effects (font (size 1.27 1.27)) (justify left))
+    )
+    (property "Footprint" "Package_DFN_QFN:Infineon_PQFN-22-15-4EP_6x5mm_P0.65mm" (at 44.45 83.82 0)
+      (effects (font (size 1.27 1.27) italic) hide)
+    )
+    (property "Datasheet" "https://www.infineon.com/dgdl/ir4301.pdf?fileId=5546d462533600a4015355d5fc691819" (at 44.45 83.82 0)
+      (effects (font (size 1.27 1.27)) hide)
+    )
+    (pin "10")
+    (pin "9")
+    (pin "5")
+    (pin "7")
+    (pin "6")
+    (pin "8")
+    (pin "4")
+    (pin "15")
+    (pin "14")
+    (pin "12")
+    (pin "2")
+    (pin "3")
+    (pin "13")
+    (pin "1")
+    (pin "11")
+    (instances
+      (project "check_in_wizard"
+        (path "/adf1bd21-a752-457d-b3de-2ef350314693"
+          (reference "U2") (unit 1)
+        )
+      )
     )
   )

Commit message: y nghia
Parts:
- added P1: RFID-RC522-MODULE, symbol rfid-rc522-module:RFID-RC522-MODULE
Changed lines of the file:
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@@
+    )
+  )
+  (symbol (lib_id "rfid-rc522-module:RFID-RC522-MODULE") (at 76.2 44.45 0) (unit 1)
+    (in_bom yes) (on_board yes) (dnp no) (fields_autoplaced)
+    (property "Reference" "P1" (at 92.71 42.545 0)
+      (effects (font (size 1.524 1.524)) (justify left))
+    )
+    (property "Value" "RFID-RC522-MODULE" (at 92.71 45.085 0)
+      (effects (font (size 1.524 1.524)) (justify left))
+    )
+    (property "Footprint" "" (at 76.2 44.45 0)
+      (effects (font (size 1.524 1.524)))
+    )
+    (property "Datasheet" "" (at 76.2 44.45 0)
+      (effects (font (size 1.524 1.524)))
+    )
+    (pin "8")
+    (pin "6")
+    (pin "7")
+    (pin "4")
+    (pin "2")
+    (pin "5")
+    (pin "1")
+    (pin "3")
+    (instances
+      (project "check_in_wizard"
+        (path "/adf1bd21-a752-457d-b3de-2ef350314693"
+          (reference "P1") (unit 1)
+        )
+      )
     )
   )

Commit message: new
Parts:
- removed U1: STM32F103C8Tx, Package_QFP:LQFP-48_7x7mm_P0.5mm, symbol MCU_ST_STM32F1:STM32F103C8Tx
- removed U2: IR4301, Package_DFN_QFN:Infineon_PQFN-22-15-4EP_6x5mm_P0.65mm, symbol Amplifier_Audio:IR4301
- added Brd1: SSD1306, symbol SSD1306-128x64_OLED:SSD1306
- added U3: YAAJ_BluePill, symbol YAAJ_BluePill:YAAJ_BluePill
Connections:
- net at P1.1 (SDA): now also U3.29 (PA4)
- net at P1.2 (SCK): now also U3.30 (PA5)
- net at P1.3 (MOSI): now also U3.32 (PA7)
- net at P1.4 (MISO): now also U3.31 (PA6)
- net at P1.6 (GND): now also U3.40 (GND)
- net at P1.7 (RST): now also P1.8 (3.3V), U3.38 (3V3)
Other:
- moved on the sheet: P1
Changed lines of the file:
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@@
 (kicad_sch (version 20230121) (generator eeschema)
   (paper "A4")
-  (symbol (lib_id "Device:Buzzer") (at 162.56 46.99 0) (unit 1)
+  (junction (at 165.1 55.88) (diameter 0) (color 0 0 0 0)
+  )
+  (wire (pts (xy 165.1 55.88) (xy 143.51 55.88))
+    (stroke (width 0) (type default))
+  )
+  (wire (pts (xy 165.1 88.9) (xy 165.1 87.63))
+    (stroke (width 0) (type default))
+  )
+  (wire (pts (xy 168.91 69.85) (xy 167.64 69.85))
+    (stroke (width 0) (type default))
+  )
+  (wire (pts (xy 165.1 87.63) (xy 161.29 87.63))
+    (stroke (width 0) (type default))
+  )
+  (wire (pts (xy 167.64 69.85) (xy 167.64 53.34))
+    (stroke (width 0) (type default))
+  )
+  (wire (pts (xy 167.64 53.34) (xy 195.58 53.34))
+    (stroke (width 0) (type default))
+  )
+  (wire (pts (xy 163.83 82.55) (xy 161.29 82.55))
+    (stroke (width 0) (type default))
+  )
+  (wire (pts (xy 168.91 80.01) (xy 161.29 80.01))
+    (stroke (width 0) (type default))
+  )
+  (wire (pts (xy 163.83 77.47) (xy 163.83 82.55))
+    (stroke (width 0) (type default))
+  )
+  (wire (pts (xy 168.91 55.88) (xy 165.1 55.88))
+    (stroke (width 0) (type default))
+  )
+  (wire (pts (xy 168.91 66.04) (xy 165.1 66.04))
+    (stroke (width 0) (type default))
+  )
+  (wire (pts (xy 161.29 85.09) (xy 168.91 85.09))
+    (stroke (width 0) (type default))
+  )
+  (wire (pts (xy 143.51 55.88) (xy 143.51 59.69))
+    (stroke (width 0) (type default))
+  )
+  (wire (pts (xy 140.97 119.38) (xy 140.97 115.57))
+    (stroke (width 0) (type default))
+  )
+  (wire (pts (xy 168.91 77.47) (xy 163.83 77.47))
+    (stroke (width 0) (type default))
+  )
+  (wire (pts (xy 168.91 88.9) (xy 165.1 88.9))
+    (stroke (width 0) (type default))
+  )
+  (wire (pts (xy 165.1 66.04) (xy 165.1 55.88))
+    (stroke (width 0) (type default))
+  )
+  (wire (pts (xy 195.58 119.38) (xy 140.97 119.38))
+    (stroke (width 0) (type default))
+  )
+  (wire (pts (xy 168.91 81.28) (xy 168.91 80.01))
+    (stroke (width 0) (type default))
+  )
+  (wire (pts (xy 195.58 53.34) (xy 195.58 119.38))
+    (stroke (width 0) (type default))
+  )
+  (wire (pts (xy 168.91 62.23) (xy 168.91 55.88))
+    (stroke (width 0) (type default))
+  )
+  (symbol (lib_id "Device:Buzzer") (at 223.52 62.23 0) (unit 1)
     (in_bom yes) (on_board yes) (dnp no) (fields_autoplaced)
-    (property "Reference" "BZ1" (at 166.37 45.72 0)
+    (property "Reference" "BZ1" (at 227.33 60.96 0)
       (effects (font (size 1.27 1.27)) (justify left))
     )
-    (property "Value" "Buzzer" (at 166.37 48.26 0)
+    (property "Value" "Buzzer" (at 227.33 63.5 0)
       (effects (font (size 1.27 1.27)) (justify left))
     )
-    (property "Footprint" "" (at 161.925 44.45 90)
+    (property "Footprint" "" (at 222.885 59.69 90)
       (effects (font (size 1.27 1.27)) hide)
     )
-    (property "Datasheet" "~" (at 161.925 44.45 90)
+    (property "Datasheet" "~" (at 222.885 59.69 90)
       (effects (font (size 1.27 1.27)) hide)
     )
@@
     )
   )
-  (symbol (lib_id "MCU_ST_STM32F1:STM32F103C8Tx") (at 138.43 100.33 0) (unit 1)
+  (symbol (lib_id "YAAJ_BluePill:YAAJ_BluePill") (at 140.97 87.63 0) (unit 1)
     (in_bom yes) (on_board yes) (dnp no) (fields_autoplaced)
-    (property "Reference" "U1" (at 143.1641 138.43 0)
+    (property "Reference" "U3" (at 143.1641 121.92 0)
       (effects (font (size 1.27 1.27)) (justify left))
     )
-    (property "Value" "STM32F103C8Tx" (at 143.1641 140.97 0)
+    (property "Value" "YAAJ_BluePill" (at 143.1641 124.46 0)
       (effects (font (size 1.27 1.27)) (justify left))
     )
-    (property "Footprint" "Package_QFP:LQFP-48_7x7mm_P0.5mm" (at 125.73 135.89 0)
-      (effects (font (size 1.27 1.27)) (justify right) hide)
-    )
-    (property "Datasheet" "https://www.st.com/resource/en/datasheet/stm32f103c8.pdf" (at 138.43 100.33 0)
+    (property "Footprint" "" (at 139.065 63.5 90)
       (effects (font (size 1.27 1.27)) hide)
     )
-    (pin "47")
+    (property "Datasheet" "" (at 139.065 63.5 90)
+      (effects (font (size 1.27 1.27)) hide)
+    )
+    (pin "10")
+    (pin "32")
+    (pin "2")
+    (pin "34")
+    (pin "36")
+    (pin "33")
+    (pin "22")
+    (pin "23")
+    (pin "19")
+    (pin "26")
+    (pin "16")
+    (pin "30")
+    (pin "27")
     (pin "3")
-    (pin "30")
+    (pin "14")
+    (pin "15")
+    (pin "28")
+    (pin "17")
+    (pin "31")
+    (pin "35")
+    (pin "25")
+    (pin "37")
+    (pin "29")
+    (pin "20")
+    (pin "21")
+    (pin "11")
+    (pin "12")
+    (pin "13")
+    (pin "18")
+    (pin "24")
+    (pin "1")
+    (pin "38")
+    (pin "39")
+    (pin "4")
     (pin "40")
-    (pin "23")
-    (pin "24")
-    (pin "31")
-    (pin "16")
-    (pin "17")
-    (pin "32")
-    (pin "41")
-    (pin "45")
-    (pin "8")
-    (pin "15")
-    (pin "22")
-    (pin "39")
-    (pin "9")
-    (pin "19")
-    (pin "2")
-    (pin "10")
-    (pin "44")
-    (pin "13")
-    (pin "34")
-    (pin "26")
-    (pin "21")
-    (pin "42")
-    (pin "29")
-    (pin "18")
-    (pin "38")
-    (pin "48")
-    (pin "14")
-    (pin "20")
-    (pin "35")
-    (pin "27")
-    (pin "12")
-    (pin "37")
-    (pin "28")
-    (pin "1")
-    (pin "33")
-    (pin "4")
-    (pin "43")
-    (pin "46")
     (pin "5")
     (pin "6")
     (pin "7")
-    (pin "36")
-    (pin "25")
-    (pin "11")
+    (pin "8")
+    (pin "9")
     (instances
       (project "check_in_wizard"
         (path "/adf1bd21-a752-457d-b3de-2ef350314693"
-          (reference "U1") (unit 1)
+          (reference "U3") (unit 1)
         )
       )
     )
   )
-  (symbol (lib_id "Amplifier_Audio:IR4301") (at 44.45 83.82 0) (unit 1)
+  (symbol (lib_id "SSD1306-128x64_OLED:SSD1306") (at 214.63 85.09 0) (unit 1)
     (in_bom yes) (on_board yes) (dnp no) (fields_autoplaced)
-    (property "Reference" "U2" (at 51.7241 60.96 0)
+    (property "Reference" "Brd1" (at 222.25 83.82 0)
       (effects (font (size 1.27 1.27)) (justify left))
     )
-    (property "Value" "IR4301" (at 51.7241 63.5 0)
+    (property "Value" "SSD1306" (at 222.25 86.36 0)
       (effects (font (size 1.27 1.27)) (justify left))
     )
-    (property "Footprint" "Package_DFN_QFN:Infineon_PQFN-22-15-4EP_6x5mm_P0.65mm" (at 44.45 83.82 0)
-      (effects (font (size 1.27 1.27) italic) hide)
-    )
-    (property "Datasheet" "https://www.infineon.com/dgdl/ir4301.pdf?fileId=5546d462533600a4015355d5fc691819" (at 44.45 83.82 0)
+    (property "Footprint" "" (at 214.63 78.74 0)
       (effects (font (size 1.27 1.27)) hide)
     )
-    (pin "10")
-    (pin "9")
-    (pin "5")
-    (pin "7")
-    (pin "6")
-    (pin "8")
+    (property "Datasheet" "" (at 214.63 78.74 0)
+      (effects (font (size 1.27 1.27)) hide)
+    )
+    (pin "1")
     (pin "4")
-    (pin "15")
-    (pin "14")
-    (pin "12")
+    (pin "3")
     (pin "2")
-    (pin "3")
-    (pin "13")
-    (pin "1")
-    (pin "11")
     (instances
       (project "check_in_wizard"
         (path "/adf1bd21-a752-457d-b3de-2ef350314693"
-          (reference "U2") (unit 1)
+          (reference "Brd1") (unit 1)
         )
       )
     )
   )
-  (symbol (lib_id "rfid-rc522-module:RFID-RC522-MODULE") (at 76.2 44.45 0) (unit 1)
-    (in_bom yes) (on_board yes) (dnp no) (fields_autoplaced)
-    (property "Reference" "P1" (at 92.71 42.545 0)
-      (effects (font (size 1.524 1.524)) (justify left))
-    )
-    (property "Value" "RFID-RC522-MODULE" (at 92.71 45.085 0)
-      (effects (font (size 1.524 1.524)) (justify left))
-    )
-    (property "Footprint" "" (at 76.2 44.45 0)
+  (symbol (lib_id "rfid-rc522-module:RFID-RC522-MODULE") (at 182.88 74.93 270) (mirror x) (unit 1)
+    (in_bom yes) (on_board yes) (dnp no)
+    (property "Reference" "P1" (at 183.515 96.52 90)
       (effects (font (size 1.524 1.524)))
     )
-    (property "Datasheet" "" (at 76.2 44.45 0)
+    (property "Value" "RFID-RC522-MODULE" (at 183.515 93.98 90)
       (effects (font (size 1.524 1.524)))
     )
+    (property "Footprint" "" (at 182.88 74.93 0)
+      (effects (font (size 1.524 1.524)))
+    )
+    (property "Datasheet" "" (at 182.88 74.93 0)
+      (effects (font (size 1.524 1.524)))
+    )

Commit message: update schematic pdf file
Connections:
- net at BZ1.1 (+): now also U3.6 (PA9)
- net at BZ1.2 (-): now also Brd1.1 (GND), P1.6 (GND), U3.40 (GND)
- net at U3.14 (PB6): now also Brd1.3 (SCL)
- net at U3.15 (PB7): now also Brd1.4 (SDA)
- net at P1.7 (RST), P1.8 (3.3V), U3.38 (3V3): now also Brd1.2 (VCC)
Other:
- title: (none) -> Class Check-in Wizard 
- moved on the sheet: BZ1, Brd1, P1
Changed lines of the file:
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@@
 (kicad_sch (version 20230121) (generator eeschema)
   (paper "A4")
-  (junction (at 165.1 55.88) (diameter 0) (color 0 0 0 0)
-  )
-  (wire (pts (xy 165.1 55.88) (xy 143.51 55.88))
-    (stroke (width 0) (type default))
-  )
-  (wire (pts (xy 165.1 88.9) (xy 165.1 87.63))
-    (stroke (width 0) (type default))
-  )
-  (wire (pts (xy 168.91 69.85) (xy 167.64 69.85))
-    (stroke (width 0) (type default))
-  )
-  (wire (pts (xy 165.1 87.63) (xy 161.29 87.63))
-    (stroke (width 0) (type default))
-  )
-  (wire (pts (xy 167.64 69.85) (xy 167.64 53.34))
-    (stroke (width 0) (type default))
-  )
-  (wire (pts (xy 167.64 53.34) (xy 195.58 53.34))
-    (stroke (width 0) (type default))
-  )
-  (wire (pts (xy 163.83 82.55) (xy 161.29 82.55))
-    (stroke (width 0) (type default))
-  )
-  (wire (pts (xy 168.91 80.01) (xy 161.29 80.01))
-    (stroke (width 0) (type default))
-  )
-  (wire (pts (xy 163.83 77.47) (xy 163.83 82.55))
-    (stroke (width 0) (type default))
-  )
-  (wire (pts (xy 168.91 55.88) (xy 165.1 55.88))
-    (stroke (width 0) (type default))
-  )
-  (wire (pts (xy 168.91 66.04) (xy 165.1 66.04))
-    (stroke (width 0) (type default))
-  )
-  (wire (pts (xy 161.29 85.09) (xy 168.91 85.09))
+  (title_block
+    (title "Class Check-in Wizard ")
+    (date "2024-02-28")
+    (rev "1")
+  )
+  (junction (at 140.97 119.38) (diameter 0) (color 0 0 0 0)
+  )
+  (junction (at 143.51 55.88) (diameter 0) (color 0 0 0 0)
+  )
+  (junction (at 82.55 86.36) (diameter 0) (color 0 0 0 0)
+  )
+  (junction (at 163.83 55.88) (diameter 0) (color 0 0 0 0)
+  )
+  (wire (pts (xy 143.51 55.88) (xy 163.83 55.88))
+    (stroke (width 0) (type default))
+  )
+  (wire (pts (xy 82.55 86.36) (xy 82.55 119.38))
+    (stroke (width 0) (type default))
+  )
+  (wire (pts (xy 106.68 55.88) (xy 143.51 55.88))
+    (stroke (width 0) (type default))
+  )
+  (wire (pts (xy 106.68 97.79) (xy 106.68 55.88))
+    (stroke (width 0) (type default))
+  )
+  (wire (pts (xy 168.91 95.25) (xy 163.83 95.25))
+    (stroke (width 0) (type default))
+  )
+  (wire (pts (xy 199.39 119.38) (xy 140.97 119.38))
+    (stroke (width 0) (type default))
+  )
+  (wire (pts (xy 166.37 87.63) (xy 166.37 80.01))
+    (stroke (width 0) (type default))
+  )
+  (wire (pts (xy 165.1 91.44) (xy 165.1 85.09))
+    (stroke (width 0) (type default))
+  )
+  (wire (pts (xy 168.91 72.39) (xy 163.83 72.39))
+    (stroke (width 0) (type default))
+  )
+  (wire (pts (xy 82.55 67.31) (xy 82.55 86.36))
+    (stroke (width 0) (type default))
+  )
+  (wire (pts (xy 199.39 60.96) (xy 199.39 119.38))
+    (stroke (width 0) (type default))
+  )
+  (wire (pts (xy 168.91 76.2) (xy 166.37 76.2))
     (stroke (width 0) (type default))
   )
@@
     (stroke (width 0) (type default))
   )
+  (wire (pts (xy 168.91 55.88) (xy 168.91 68.58))
+    (stroke (width 0) (type default))
+  )
+  (wire (pts (xy 163.83 95.25) (xy 163.83 87.63))
+    (stroke (width 0) (type default))
+  )
+  (wire (pts (xy 165.1 82.55) (xy 161.29 82.55))
+    (stroke (width 0) (type default))
+  )
   (wire (pts (xy 140.97 119.38) (xy 140.97 115.57))
     (stroke (width 0) (type default))
   )
-  (wire (pts (xy 168.91 77.47) (xy 163.83 77.47))
-    (stroke (width 0) (type default))
-  )
-  (wire (pts (xy 168.91 88.9) (xy 165.1 88.9))
-    (stroke (width 0) (type default))
-  )
-  (wire (pts (xy 165.1 66.04) (xy 165.1 55.88))
-    (stroke (width 0) (type default))
-  )
-  (wire (pts (xy 195.58 119.38) (xy 140.97 119.38))
-    (stroke (width 0) (type default))
-  )
-  (wire (pts (xy 168.91 81.28) (xy 168.91 80.01))
-    (stroke (width 0) (type default))
-  )
-  (wire (pts (xy 195.58 53.34) (xy 195.58 119.38))
-    (stroke (width 0) (type default))
-  )
-  (wire (pts (xy 168.91 62.23) (xy 168.91 55.88))
-    (stroke (width 0) (type default))
-  )
-  (symbol (lib_id "Device:Buzzer") (at 223.52 62.23 0) (unit 1)
+  (wire (pts (xy 116.84 67.31) (xy 82.55 67.31))
+    (stroke (width 0) (type default))
+  )
+  (wire (pts (xy 116.84 74.93) (xy 116.84 67.31))
+    (stroke (width 0) (type default))
+  )
+  (wire (pts (xy 163.83 87.63) (xy 161.29 87.63))
+    (stroke (width 0) (type default))
+  )
+  (wire (pts (xy 116.84 80.01) (xy 120.65 80.01))
+    (stroke (width 0) (type default))
+  )
+  (wire (pts (xy 102.87 102.87) (xy 120.65 102.87))
+    (stroke (width 0) (type default))
+  )
+  (wire (pts (xy 102.87 100.33) (xy 120.65 100.33))
+    (stroke (width 0) (type default))
+  )
+  (wire (pts (xy 168.91 91.44) (xy 165.1 91.44))
+    (stroke (width 0) (type default))
+  )
+  (wire (pts (xy 168.91 87.63) (xy 166.37 87.63))
+    (stroke (width 0) (type default))
+  )
+  (wire (pts (xy 102.87 95.25) (xy 102.87 86.36))
+    (stroke (width 0) (type default))
+  )
+  (wire (pts (xy 165.1 85.09) (xy 161.29 85.09))
+    (stroke (width 0) (type default))
+  )
+  (wire (pts (xy 166.37 60.96) (xy 199.39 60.96))
+    (stroke (width 0) (type default))
+  )
+  (wire (pts (xy 166.37 76.2) (xy 166.37 60.96))
+    (stroke (width 0) (type default))
+  )
+  (wire (pts (xy 82.55 119.38) (xy 140.97 119.38))
+    (stroke (width 0) (type default))
+  )
+  (wire (pts (xy 102.87 86.36) (xy 82.55 86.36))
+    (stroke (width 0) (type default))
+  )
+  (wire (pts (xy 102.87 97.79) (xy 106.68 97.79))
+    (stroke (width 0) (type default))
+  )
+  (wire (pts (xy 166.37 80.01) (xy 161.29 80.01))
+    (stroke (width 0) (type default))
+  )
+  (wire (pts (xy 163.83 72.39) (xy 163.83 55.88))
+    (stroke (width 0) (type default))
+  )
+  (wire (pts (xy 165.1 83.82) (xy 165.1 82.55))
+    (stroke (width 0) (type default))
+  )
+  (wire (pts (xy 163.83 55.88) (xy 168.91 55.88))
+    (stroke (width 0) (type default))
+  )
+  (wire (pts (xy 168.91 83.82) (xy 165.1 83.82))
+    (stroke (width 0) (type default))
+  )
+  (symbol (lib_id "Device:Buzzer") (at 114.3 77.47 180) (unit 1)
     (in_bom yes) (on_board yes) (dnp no) (fields_autoplaced)
-    (property "Reference" "BZ1" (at 227.33 60.96 0)
-      (effects (font (size 1.27 1.27)) (justify left))
-    )
-    (property "Value" "Buzzer" (at 227.33 63.5 0)
-      (effects (font (size 1.27 1.27)) (justify left))
-    )
-    (property "Footprint" "" (at 222.885 59.69 90)
-      (effects (font (size 1.27 1.27)) hide)
-    )
-    (property "Datasheet" "~" (at 222.885 59.69 90)
+    (property "Reference" "BZ1" (at 113.5449 69.85 0)
+      (effects (font (size 1.27 1.27)))
+    )
+    (property "Value" "Buzzer" (at 113.5449 72.39 0)
+      (effects (font (size 1.27 1.27)))
+    )
+    (property "Footprint" "" (at 114.935 80.01 90)
+      (effects (font (size 1.27 1.27)) hide)
+    )
+    (property "Datasheet" "~" (at 114.935 80.01 90)
       (effects (font (size 1.27 1.27)) hide)
     )
@@
     )
   )
-  (symbol (lib_id "SSD1306-128x64_OLED:SSD1306") (at 214.63 85.09 0) (unit 1)
+  (symbol (lib_id "SSD1306-128x64_OLED:SSD1306") (at 93.98 99.06 270) (unit 1)
     (in_bom yes) (on_board yes) (dnp no) (fields_autoplaced)
-    (property "Reference" "Brd1" (at 222.25 83.82 0)
-      (effects (font (size 1.27 1.27)) (justify left))
-    )
-    (property "Value" "SSD1306" (at 222.25 86.36 0)
-      (effects (font (size 1.27 1.27)) (justify left))
-    )
-    (property "Footprint" "" (at 214.63 78.74 0)
-      (effects (font (size 1.27 1.27)) hide)
-    )
-    (property "Datasheet" "" (at 214.63 78.74 0)
+    (property "Reference" "Brd1" (at 93.98 87.63 90)
+      (effects (font (size 1.27 1.27)))
+    )
+    (property "Value" "SSD1306" (at 93.98 90.17 90)
+      (effects (font (size 1.27 1.27)))
+    )
+    (property "Footprint" "" (at 100.33 99.06 0)
+      (effects (font (size 1.27 1.27)) hide)
+    )
+    (property "Datasheet" "" (at 100.33 99.06 0)
       (effects (font (size 1.27 1.27)) hide)
     )
@@
     )
   )
-  (symbol (lib_id "rfid-rc522-module:RFID-RC522-MODULE") (at 182.88 74.93 270) (mirror x) (unit 1)
+  (symbol (lib_id "rfid-rc522-module:RFID-RC522-MODULE") (at 182.88 81.28 270) (mirror x) (unit 1)
     (in_bom yes) (on_board yes) (dnp no)
-    (property "Reference" "P1" (at 183.515 96.52 90)
-      (effects (font (size 1.524 1.524)))
-    )
-    (property "Value" "RFID-RC522-MODULE" (at 183.515 93.98 90)
-      (effects (font (size 1.524 1.524)))
-    )
-    (property "Footprint" "" (at 182.88 74.93 0)
-      (effects (font (size 1.524 1.524)))
-    )
-    (property "Datasheet" "" (at 182.88 74.93 0)
-      (effects (font (size 1.524 1.524)))
-    )
+    (property "Reference" "P1" (at 183.515 102.87 90)
+      (effects (font (size 1.524 1.524)))
+    )
+    (property "Value" "RFID-RC522-MODULE" (at 183.515 100.33 90)
+      (effects (font (size 1.524 1.524)))
+    )
+    (property "Footprint" "" (at 182.88 81.28 0)
+      (effects (font (size 1.524 1.524)))
+    )
+    (property "Datasheet" "" (at 182.88 81.28 0)
+      (effects (font (size 1.524 1.524)))
+    )

Commit message: Homework 3 updated
Parts:
- renumbered Brd1 to OLED
Changed lines of the file:
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@@
   )
   (symbol (lib_id "SSD1306-128x64_OLED:SSD1306") (at 93.98 99.06 270) (unit 1)
-    (in_bom yes) (on_board yes) (dnp no) (fields_autoplaced)
-    (property "Reference" "Brd1" (at 93.98 87.63 90)
+    (in_bom yes) (on_board yes) (dnp no)
+    (property "Reference" "OLED" (at 93.98 87.63 90)
       (effects (font (size 1.27 1.27)))
     )
@@
       (project "check_in_wizard"
         (path "/adf1bd21-a752-457d-b3de-2ef350314693"
-          (reference "Brd1") (unit 1)
+          (reference "OLED") (unit 1)
         )
       )
